Commit message: driver and demo updates

File: rm_65_description/urdf/rm_65.urdf.xacro (robot description, xacro)
@@ -1,29 +1,23 @@
-<?xml version="1.0" ?>
-<robot name="rm_65" xmlns:xacro="http://www.ros.org/wiki/xacro">
+<?xml version="1.0" encoding="utf-8"?>
+<robot  name="rm_65" xmlns:xacro="http://www.ros.org/wiki/xacro">
 <xacro:include filename="$(find rm_65_description)/urdf/rm_65.transmission.xacro"/>
 <xacro:include filename="$(find rm_65_description)/urdf/rm_65.gazebo.xacro"/>
-<!-- <xacro:include filename="$(find rm_65_description)/urdf/common.gazebo.xacro"/> -->
-<!-- Inertial matrix -->
-<xacro:macro name="inertial_matrix" params="mass">
-<inertial>
-    <mass value="${mass}" />
-    <inertia ixx="1.0" ixy="0.0" ixz="0.0" iyy="0.5" iyz="0.0" izz="1.0" />
-</inertial>
-</xacro:macro>
+  <link name="dummy">
+  </link>
   <link
     name="base_link">
     <inertial>
       <origin
-        xyz="0.000364099338239377 -0.000180492589223954 0.0523748178864983"
+        xyz="-0.000433277303987328 -3.54664423471128E-05 0.0599427668933796"
         rpy="0 0 0" />
       <mass
         value="14" />
       <inertia
-        ixx="0.000737277875726733"
-        ixy="1.52768076655905E-06"
-        ixz="-1.75138967359717E-05"
-        iyy="0.000723643543181375"
-        iyz="-8.08320706906158E-07"
-        izz="0.000487026166065825" />
+        ixx="0.0017261110801622"
+        ixy="2.52746264980217E-06"
+        ixz="-3.67690303614961E-05"
+        iyy="0.00170987405835604"
+        iyz="1.67996364994424E-06"
+        izz="0.000904023422915791" />
     </inertial>
     <visual>
@@ -57,41 +51,45 @@
     <kd value="1.0"/>
   </gazebo>
+  <joint name="dummy_joint" type="fixed">
+    <parent link="dummy" />
+    <child link="base_link" />
+  </joint>
   <link
     name="Link1">
     <inertial>
       <origin
-        xyz="-1.79862733952242E-05 -0.0216004812887538 0.0719258896443856"
-        rpy="0 0 0" />
-      <mass
-        value="0.200843839724735" />
-      <inertia
-        ixx="0.000531136984021332"
-        ixy="-4.32776127280478E-07"
-        ixz="1.04793272362077E-06"
-        iyy="0.000497444611373595"
-        iyz="0.000106254355496355"
-        izz="0.000282103590137435" />
-    </inertial>
-    <visual>
-      <origin
-        xyz="0 0 0"
-        rpy="0 0 0" />
-      <geometry>
-        <mesh
-          filename="package://rm_65_description/meshes/Link1.STL" />
-      </geometry>
-      <material
-        name="">
-        <color
-          rgba="1 1 1 1" />
-      </material>
-    </visual>
-    <collision>
-      <origin
-        xyz="0 0 0"
-        rpy="0 0 0" />
-      <geometry>
-        <mesh
-          filename="package://rm_65_description/meshes/Link1.STL" />
+        xyz="1.2226305431569E-08 0.0211079974844683 -0.0251854220842269"
+        rpy="0 0 0" />
+      <mass
+        value="0.593563443690403" />
+      <inertia
+        ixx="0.00126614120341847"
+        ixy="-1.294980943835E-08"
+        ixz="-9.80120923066996E-09"
+        iyy="0.00118168178300364"
+        iyz="-0.00021121727444415"
+        izz="0.00056135241627747" />
+    </inertial>
+    <visual>
+      <origin
+        xyz="0 0 0"
+        rpy="0 0 0" />
+      <geometry>
+        <mesh
+          filename="package://rm_65_description/meshes/link1.STL" />
+      </geometry>
+      <material
+        name="">
+        <color
+          rgba="1 1 1 1" />
+      </material>
+    </visual>
+    <collision>
+      <origin
+        xyz="0 0 0"
+        rpy="0 0 0" />
+      <geometry>
+        <mesh
+          filename="package://rm_65_description/meshes/link1.STL" />
       </geometry>
     </collision>
@@ -101,6 +99,6 @@
     type="revolute">
     <origin
-      xyz="0.00019414 0.0001 0.138"
-      rpy="-2.3944E-16 0 3.1416" />
+      xyz="0 0 0.2405"
+      rpy="0 0 0" />
     <parent
       link="base_link" />
@@ -110,7 +108,7 @@
       xyz="0 0 1" />
     <limit
-      lower="-3.14"
-      upper="3.14"
-      effort="300"
+      lower="-3.1"
+      upper="3.1"
+      effort="60"
       velocity="3.14" />
 	<dynamics damping="50" friction="1"/>
@@ -120,37 +118,37 @@
     <inertial>
       <origin
-        xyz="0.133181684940056 -4.09216469913973E-05 0.0184216581306229"
-        rpy="0 0 0" />
-      <mass
-        value="0.321307361964397" />
-      <inertia
-        ixx="0.000440014028766832"
-        ixy="5.6579315252598E-07"
-        ixz="-0.000654853772254918"
-        iyy="0.00298539844077015"
-        iyz="1.20748806355071E-07"
-        izz="0.00284806640328522" />
-    </inertial>
-    <visual>
-      <origin
-        xyz="0 0 0"
-        rpy="0 0 0" />
-      <geometry>
-        <mesh
-          filename="package://rm_65_description/meshes/Link2.STL" />
-      </geometry>
-      <material
-        name="">
-        <color
-          rgba="1 1 1 1" />
-      </material>
-    </visual>
-    <collision>
-      <origin
-        xyz="0 0 0"
-        rpy="0 0 0" />
-      <geometry>
-        <mesh
-          filename="package://rm_65_description/meshes/Link2.STL" />
+        xyz="0.152256463426163 4.75383656106654E-07 -0.00620260383607792"
+        rpy="0 0 0" />
+      <mass
+        value="0.864175046869043" />
+      <inertia
+        ixx="0.00089150298478414"
+        ixy="-2.23268489334765E-08"
+        ixz="0.00156246461035015"
+        iyy="0.00733754343083901"
+        iyz="6.28110889329165E-09"
+        izz="0.00697869103915473" />
+    </inertial>
+    <visual>
+      <origin
+        xyz="0 0 0"
+        rpy="0 0 0" />
+      <geometry>
+        <mesh
+          filename="package://rm_65_description/meshes/link2.STL" />
+      </geometry>
+      <material
+        name="">
+        <color
+          rgba="1 1 1 1" />
+      </material>
+    </visual>
+    <collision>
+      <origin
+        xyz="0 0 0"
+        rpy="0 0 0" />
+      <geometry>
+        <mesh
+          filename="package://rm_65_description/meshes/link2.STL" />
       </geometry>
     </collision>
@@ -160,5 +158,5 @@
     type="revolute">
     <origin
-      xyz="0 0.016171 0.1012"
+      xyz="0 0 0"
       rpy="1.5708 -1.5708 0" />
     <parent
@@ -167,9 +165,9 @@
       link="Link2" />
     <axis
-      xyz="0 0 -1" />
-    <limit
-      lower="-2.269"
-      upper="2.269"
-      effort="300"
+      xyz="0 0 1" />
+    <limit
+      lower="-2.268"
+      upper="2.268"
+      effort="60"
       velocity="3.14" />
 	<dynamics damping="50" friction="1"/>
@@ -179,37 +177,37 @@
     <inertial>
       <origin
-        xyz="-3.56690328818382E-06 -0.0512866037910138 2.10951876323563E-05"
-        rpy="0 0 0" />
-      <mass
-        value="0.102772515618803" />
-      <inertia
-        ixx="0.000236471825455939"
-        ixy="-2.85439143488268E-09"
-        ixz="-4.04883470632046E-10"
-        iyy="7.36858171850124E-05"
-        iyz="5.2218422744868E-05"
-        izz="0.000233873582444284" />
-    </inertial>
-    <visual>
-      <origin
-        xyz="0 0 0"
-        rpy="0 0 0" />
-      <geometry>
-        <mesh
-          filename="package://rm_65_description/meshes/Link3.STL" />
-      </geometry>
-      <material
-        name="">
-        <color
-          rgba="1 1 1 1" />
-      </material>
-    </visual>
-    <collision>
-      <origin
-        xyz="0 0 0"
-        rpy="0 0 0" />
-      <geometry>
-        <mesh
-          filename="package://rm_65_description/meshes/Link3.STL" />
+        xyz="5.05312670989961E-06 -0.0595925663694732 0.010569069212336"
+        rpy="0 0 0" />
+      <mass
+        value="0.289633681624654" />
+      <inertia
+        ixx="0.00063737100450158"
+        ixy="-7.05261293649751E-08"
+        ixz="-3.86643272239426E-08"
+        iyy="0.00015648388095025"
+        iyz="-0.00014461035994916"
+        izz="0.000614178164773085" />
+    </inertial>
+    <visual>
+      <origin
+        xyz="0 0 0"
+        rpy="0 0 0" />
+      <geometry>
+        <mesh
+          filename="package://rm_65_description/meshes/link3.STL" />
+      </geometry>
+      <material
+        name="">
+        <color
+          rgba="1 1 1 1" />
+      </material>
+    </visual>
+    <collision>
+      <origin
+        xyz="0 0 0"
+        rpy="0 0 0" />
+      <geometry>
+        <mesh
+          filename="package://rm_65_description/meshes/link3.STL" />
       </geometry>
     </collision>
@@ -219,6 +217,6 @@
     type="revolute">
     <origin
-      xyz="0.25576 0 0.0035251"
-      rpy="1.1972E-16 1.4979E-28 1.5708" />
+      xyz="0.256 0 0"
+      rpy="0 0 1.5708" />
     <parent
       link="Link2" />
@@ -226,10 +224,10 @@
       link="Link3" />
     <axis
-      xyz="0 0 -1" />
-    <limit
-      lower="-2.356"
-      upper="2.356"
-      effort="300"
-      velocity="3.14" />
+      xyz="0 0 1" />
+    <limit
+      lower="-2.355"
+      upper="2.355"
+      effort="30"
+      velocity="3.92" />
 	<dynamics damping="50" friction="1"/>
   </joint>
@@ -238,37 +236,37 @@
     <inertial>
       <origin
-        xyz="6.79143687717758E-05 0.0172073813582943 0.0550497562490089"
-        rpy="0 0 0" />
-      <mass
-        value="0.0751534548575527" />
-      <inertia
-        ixx="0.000114971629184183"
-        ixy="1.55043636696422E-08"
-        ixz="2.03173541830271E-07"
-        iyy="0.000105991655073516"
-        iyz="-2.1400189980959E-05"
-        izz="5.71243912493456E-05" />
-    </inertial>
-    <visual>
-      <origin
-        xyz="0 0 0"
-        rpy="0 0 0" />
-      <geometry>
-        <mesh
-          filename="package://rm_65_description/meshes/Link4.STL" />
-      </geometry>
-      <material
-        name="">
-        <color
-          rgba="1 1 1 1" />
-      </material>
-    </visual>
-    <collision>
-      <origin
-        xyz="0 0 0"
-        rpy="0 0 0" />
-      <geometry>
-        <mesh
-          filename="package://rm_65_description/meshes/Link4.STL" />
+        xyz="1.15516617405898E-06 -0.0180424468598241 -0.0215394748352687"
+        rpy="0 0 0" />
+      <mass
+        value="0.239419768320061" />
+      <inertia
+        ixx="0.000285938919722783"
+        ixy="3.07101359163101E-09"
+        ixz="-2.21994118981953E-09"
+        iyy="0.000262727540304212"
+        iyz="4.4236583260078E-05"
+        izz="0.000119888082791859" />
+    </inertial>
+    <visual>
+      <origin
+        xyz="0 0 0"
+        rpy="0 0 0" />
+      <geometry>
+        <mesh
+          filename="package://rm_65_description/meshes/link4.STL" />
+      </geometry>
+      <material
+        name="">
+        <color
+          rgba="1 1 1 1" />
+      </material>
+    </visual>
+    <collision>
+      <origin
+        xyz="0 0 0"
+        rpy="0 0 0" />
+      <geometry>
+        <mesh
+          filename="package://rm_65_description/meshes/link4.STL" />
       </geometry>
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