Commit message: doc: fix eco63 gazebo error

File: rm_description/urdf/ECO63/rm_eco63.urdf.xacro (robot description, xacro)
@@ -141,6 +141,9 @@
       lower="-3.1"
       upper="3.1"
-      effort="0"
+      effort="100"
       velocity="0" />
+      <dynamics
+      damping="50"
+      friction="1" />
   </joint>
   <link
@@ -199,6 +202,9 @@
       lower="-3.1"
       upper="3.1"
-      effort="0"
-      velocity="0" />
+      effort="100"
+      velocity="1" />
+      <dynamics
+      damping="50"
+      friction="1" />
   </joint>
   <link
@@ -257,6 +263,9 @@
       lower="-2.95"
       upper="2.76"
-      effort="0"
-      velocity="0" />
+      effort="100"
+      velocity="1" />
+    <dynamics
+      damping="50"
+      friction="1" />
   </joint>
   <link
@@ -315,6 +324,9 @@
       lower="-2.44"
       upper="2.44"
-      effort="0"
-      velocity="0" />
+      effort="100"
+      velocity="1" />
+    <dynamics
+      damping="50"
+      friction="1" />
   </joint>
   <link
@@ -373,6 +385,9 @@
       lower="-3.14"
       upper="3.14"
-      effort="0"
-      velocity="0" />
+      effort="100"
+      velocity="1" />
+    <dynamics
+      damping="50"
+      friction="1" />
   </joint>
   <link
@@ -385,10 +400,10 @@
         value="0.080797" />
       <inertia
-        ixx="2.4449E-05"
-        ixy="-1.2142E-06"
-        ixz="-1.0223E-07"
-        iyy="2.3012E-05"
-        iyz="6.5765E-08"
-        izz="3.661E-05" />
+        ixx="0"
+        ixy="0"
+        ixz="0"
+        iyy="0"
+        iyz="0"
+        izz="0" />
     </inertial>
     <visual>
@@ -431,6 +446,9 @@
       lower="-6.28"
       upper="6.28"
-      effort="0"
-      velocity="0" />
+      effort="100"
+      velocity="1" />
+    <dynamics
+      damping="50"
+      friction="1" />
   </joint>
     <!-- Transmissions for ROS Control -->
