Commit message: doc:添加一体化六维力适配，添加控制器1.6.7适配，添加UDP控制功能适配

File: rm_description/urdf/ECO63/eco63.urdf (robot description, URDF)
Before this commit: robot rm_eco63, 7 links, 6 joints
Links:
- link Link1: mass 0.7339 -> 0.656374618338142
- link Link2: mass 1.9492 -> 5.26262523683375
- link Link3: mass 1.4553 -> 1.3509329667983
- link Link4: mass 0.27261 -> 0.733001235394853
- link Link5: mass 0.31149 -> 0.911747774463918
- link Link6: mass 0.080797 -> 0.065035417997418
- link base_link: mass 0.70684 -> 8.97974481667473
Joints:
- joint joint1: axis 0 0 1 -> 0 0 -1; limit lower=-3.1 upper=3.1 effort=0 velocity=0 -> lower=-3.105 upper=3.105 effort=60 velocity=3.14
- joint joint2: axis 0 0 1 -> 0 0 -1; limit lower=-3.1 upper=3.1 effort=0 velocity=0 -> lower=-3.105 upper=2.355 effort=60 velocity=3.14; origin xyz=-0.086 0 0 rpy=-1.5708 -1.5708 0 -> xyz=-0.086 0 0 rpy=1.5708 -1.5708 0
- joint joint3: axis 0 0 1 -> -0.0087265 0 0.99996; limit lower=-2.95 upper=2.76 effort=0 velocity=0 -> lower=-2.93 upper=2.756 effort=30 velocity=3.14; origin xyz=0.41 0 0 rpy=0 0 0 -> xyz=0.41 0 0 rpy=3.1416 -0.0087266 0
- joint joint4: limit lower=-2.44 upper=2.44 effort=0 velocity=0 -> lower=-3.105 upper=3.105 effort=10 velocity=3.14; origin xyz=0.38 0 -0.0589 rpy=0 0 1.5708 -> xyz=0.38049 0 -0.054981 rpy=-0.0087266 0 1.5708
- joint joint5: axis 0 0 1 -> 0 0 -1; limit lower=-3.14 upper=3.14 effort=0 velocity=0 -> lower=-3.105 upper=3.105 effort=10 velocity=3.14; origin xyz=0 -0.11 0 rpy=1.5708 0 0 -> xyz=0 -0.11 -0.0006 rpy=1.5708 0 0
- joint joint6: axis 0 0 1 -> 0 0 -1; limit lower=-6.28 upper=6.28 effort=0 velocity=0 -> lower=-6.28 upper=6.28 effort=10 velocity=3.14; origin xyz=0 0.079501 0 rpy=-1.5708 0 0 -> xyz=-0.00010641 0.0797 -0.00010731 rpy=-1.5708 0 0

File: rm_description/urdf/ECO63/rm_eco63.urdf.xacro (robot description, xacro)
@@ -50,15 +50,15 @@
     <inertial>
       <origin
-        xyz="0.00039308 -8.9311E-05 0.050351"
-        rpy="0 0 0" />
-      <mass
-        value="0.70684" />
-      <inertia
-        ixx="0.001114"
-        ixy="3.3208E-06"
-        ixz="-2.5536E-05"
-        iyy="0.0011138"
-        iyz="1.4832E-06"
-        izz="0.00075793" />
+        xyz="-0.0819699961303711 -0.0464753726622393 0.526722271495911"
+        rpy="0 0 0" />
+      <mass
+        value="8.97974481667473" />
+      <inertia
+        ixx="0.862297666639592"
+        ixy="-0.00170110773340804"
+        ixz="0.0134260863948258"
+        iyy="0.853404080505364"
+        iyz="-0.0335323790979435"
+        izz="0.021909948868005" />
     </inertial>
     <visual>
@@ -73,5 +73,5 @@
         name="">
         <color
-          rgba="0.79216 0.81961 0.93333 1" />
+          rgba="0.792156862745098 0.819607843137255 0.933333333333333 1" />
       </material>
     </visual>
@@ -90,15 +90,15 @@
     <inertial>
       <origin
-        xyz="-0.032161 -0.002588 -0.0071715"
-        rpy="0 0 0" />
-      <mass
-        value="0.7339" />
-      <inertia
-        ixx="0.00065754"
-        ixy="-0.00012029"
-        ixz="0.00016575"
-        iyy="0.0018838"
-        iyz="1.5479E-05"
-        izz="0.0017351" />
+        xyz="-0.0309493055609114 -0.0012728567226139 -0.00524336672353307"
+        rpy="0 0 0" />
+      <mass
+        value="0.656374618338142" />
+      <inertia
+        ixx="0.000538922068295209"
+        ixy="-6.49558484347273E-05"
+        ixz="0.000104084843141859"
+        iyy="0.00162201405585815"
+        iyz="6.13990176963193E-06"
+        izz="0.00151559483136641" />
     </inertial>
     <visual>
@@ -113,5 +113,5 @@
         name="">
         <color
-          rgba="0.79216 0.81961 0.93333 1" />
+          rgba="0.792156862745098 0.819607843137255 0.933333333333333 1" />
       </material>
     </visual>
@@ -137,255 +137,255 @@
       link="Link1" />
     <axis
+      xyz="0 0 -1" />
+    <limit
+      lower="-3.105"
+      upper="3.105"
+      effort="60"
+      velocity="3.14" />
+      <dynamics
+      damping="50"
+      friction="1" />
+  </joint>
+  <link
+    name="Link2">
+    <inertial>
+      <origin
+        xyz="0.194682247033962 -1.86346038127949E-07 0.0708742731440949"
+        rpy="0 0 0" />
+      <mass
+        value="5.26262523683375" />
+      <inertia
+        ixx="0.00404170032131906"
+        ixy="-5.65174393111021E-07"
+        ixz="0.00121807022294723"
+        iyy="0.109727764384232"
+        iyz="-2.72124756899763E-09"
+        izz="0.110681578185881" />
+    </inertial>
+    <visual>
+      <origin
+        xyz="0 0 0"
+        rpy="0 0 0" />
+      <geometry>
+        <mesh
+          filename="package://rm_description/meshes/ECO63/Link2.STL" />
+      </geometry>
+      <material
+        name="">
+        <color
+          rgba="0.866666666666667 0.866666666666667 0.890196078431372 1" />
+      </material>
+    </visual>
+    <collision>
+      <origin
+        xyz="0 0 0"
+        rpy="0 0 0" />
+      <geometry>
+        <mesh
+          filename="package://rm_description/meshes/ECO63/Link2.STL" />
+      </geometry>
+    </collision>
+  </link>
+  <joint
+    name="joint2"
+    type="revolute">
+    <origin
+      xyz="-0.086 0 0"
+      rpy="1.5708 -1.5708 0" />
+    <parent
+      link="Link1" />
+    <child
+      link="Link2" />
+    <axis
+      xyz="0 0 -1" />
+    <limit
+      lower="-3.105"
+      upper="2.355"
+      effort="60"
+      velocity="3.14" />
+      <dynamics
+      damping="50"
+      friction="1" />
+  </joint>
+  <link
+    name="Link3">
+    <inertial>
+      <origin
+        xyz="0.179310475039839 1.86928912626616E-09 0.0308638630867258"
+        rpy="0 0 0" />
+      <mass
+        value="1.3509329667983" />
+      <inertia
+        ixx="0.000796925531981305"
+        ixy="-2.89740446981148E-08"
+        ixz="-0.000607432295339128"
+        iyy="0.0219803140031169"
+        iyz="1.84171394643915E-08"
+        izz="0.022157190260175" />
+    </inertial>
+    <visual>
+      <origin
+        xyz="0 0 0"
+        rpy="0 0 0" />
+      <geometry>
+        <mesh
+          filename="package://rm_description/meshes/ECO63/Link3.STL" />
+      </geometry>
+      <material
+        name="">
+        <color
+          rgba="0.792156862745098 0.819607843137255 0.933333333333333 1" />
+      </material>
+    </visual>
+    <collision>
+      <origin
+        xyz="0 0 0"
+        rpy="0 0 0" />
+      <geometry>
+        <mesh
+          filename="package://rm_description/meshes/ECO63/Link3.STL" />
+      </geometry>
+    </collision>
+  </link>
+  <joint
+    name="joint3"
+    type="revolute">
+    <origin
+      xyz="0.41 0 0"
+      rpy="3.1416 -0.0087266 0" />
+    <parent
+      link="Link2" />
+    <child
+      link="Link3" />
+    <axis
+      xyz="-0.0087265 0 0.99996" />
+    <limit
+      lower="-2.93"
+      upper="2.756"
+      effort="30"
+      velocity="3.14" />
+      <dynamics
+      damping="50"
+      friction="1" />
+  </joint>
+  <link
+    name="Link4">
+    <inertial>
+      <origin
+        xyz="1.18737948139047E-06 -0.00995387687025817 0.0129236518197595"
+        rpy="0 0 0" />
+      <mass
+        value="0.733001235394853" />
+      <inertia
+        ixx="0.000641256799113762"
+        ixy="7.16323347889126E-09"
+        ixz="-6.76890724051393E-09"
+        iyy="0.000512473473605366"
+        iyz="-0.000109077537111131"
+        izz="0.000460316607732565" />
+    </inertial>
+    <visual>
+      <origin
+        xyz="0 0 0"
+        rpy="0 0 0" />
+      <geometry>
+        <mesh
+          filename="package://rm_description/meshes/ECO63/Link4.STL" />
+      </geometry>
+      <material
+        name="">
+        <color
+          rgba="0.866666666666667 0.866666666666667 0.890196078431372 1" />
+      </material>
+    </visual>
+    <collision>
+      <origin
+        xyz="0 0 0"
+        rpy="0 0 0" />
+      <geometry>
+        <mesh
+          filename="package://rm_description/meshes/ECO63/Link4.STL" />
+      </geometry>
+    </collision>
+  </link>
+  <joint
+    name="joint4"
+    type="revolute">
+    <origin
+      xyz="0.38049 0 -0.054981"
+      rpy="-0.0087266 0 1.5708" />
+    <parent
+      link="Link3" />
+    <child
+      link="Link4" />
+    <axis
       xyz="0 0 1" />
     <limit
-      lower="-3.1"
-      upper="3.1"
-      effort="100"
-      velocity="1" />
-      <dynamics
-      damping="50"
-      friction="1" />
-  </joint>
-  <link
-    name="Link2">
-    <inertial>
-      <origin
-        xyz="0.19469 6.6139E-07 -0.070874"
-        rpy="0 0 0" />
-      <mass
-        value="1.9492" />
-      <inertia
-        ixx="0.001497"
-        ixy="1.4887E-07"
-        ixz="-0.00045122"
-        iyy="0.040644"
-        iyz="1.3757E-08"
-        izz="0.040997" />
-    </inertial>
-    <visual>
-      <origin
-        xyz="0 0 0"
-        rpy="0 0 0" />
-      <geometry>
-        <mesh
-          filename="package://rm_description/meshes/ECO63/Link2.STL" />
-      </geometry>
-      <material
-        name="">
-        <color
-          rgba="0.79216 0.81961 0.93333 1" />
-      </material>
-    </visual>
-    <collision>
-      <origin
-        xyz="0 0 0"
-        rpy="0 0 0" />
-      <geometry>
-        <mesh
-          filename="package://rm_description/meshes/ECO63/Link2.STL" />
-      </geometry>
-    </collision>
-  </link>
-  <joint
-    name="joint2"
-    type="revolute">
-    <origin
-      xyz="-0.086 0 0"
-      rpy="-1.5708 -1.5708 0" />
-    <parent
-      link="Link1" />
-    <child
-      link="Link2" />
-    <axis
-      xyz="0 0 1" />
-    <limit
-      lower="-3.1"
-      upper="3.1"
-      effort="100"
-      velocity="1" />
-      <dynamics
-      damping="50"
-      friction="1" />
-  </joint>
-  <link
-    name="Link3">
-    <inertial>
-      <origin
-        xyz="0.1718 6.3595E-07 0.026691"
-        rpy="0 0 0" />
-      <mass
-        value="1.4553" />
-      <inertia
-        ixx="0.00094612"
-        ixy="-1.1572E-07"
-        ixz="-0.0008623"
-        iyy="0.025574"
-        iyz="-2.426E-08"
-        izz="0.025646" />
-    </inertial>
-    <visual>
-      <origin
-        xyz="0 0 0"
-        rpy="0 0 0" />
-      <geometry>
-        <mesh
-          filename="package://rm_description/meshes/ECO63/Link3.STL" />
-      </geometry>
-      <material
-        name="">
-        <color
-          rgba="0.79216 0.81961 0.93333 1" />
-      </material>
-    </visual>
-    <collision>
-      <origin
-        xyz="0 0 0"
-        rpy="0 0 0" />
-      <geometry>
-        <mesh
-          filename="package://rm_description/meshes/ECO63/Link3.STL" />
-      </geometry>
-    </collision>
-  </link>
-  <joint
-    name="joint3"
-    type="revolute">
-    <origin
-      xyz="0.41 0 0"
-      rpy="0 0 0" />
-    <parent
-      link="Link2" />
-    <child
-      link="Link3" />
-    <axis
-      xyz="0 0 1" />
-    <limit
-      lower="-2.95"
-      upper="2.76"
-      effort="100"
-      velocity="1" />
-    <dynamics
-      damping="50"
-      friction="1" />
-  </joint>
-  <link
-    name="Link4">
-    <inertial>
-      <origin
-        xyz="6.6185E-07 -0.0098798 0.013446"
-        rpy="0 0 0" />
-      <mass
-        value="0.27261" />
-      <inertia
-        ixx="0.00023835"
-        ixy="2.6006E-09"
-        ixz="-2.5717E-09"
-        iyy="0.00019072"
-        iyz="-4.0013E-05"
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
File: rm_description/urdf/GEN72/GEN72.urdf (robot description, URDF)
Before this commit: robot GEN72, 8 links, 7 joints
Links:
- link Link1: mass 0.511231576042974 -> 0.511231574249026
- link Link2: mass 0.551907023014854 -> 0.551907049708684
- link Link3: mass 0.774130450031718 -> 0.774130504869361
- link Link4: mass 0.437130215853825 -> 0.437130215851277
- link Link5: mass 0.424276753764529 -> 0.424276753764533
- link Link6: mass 0.302793039332829 -> 0.302793071336592
- link Link7: mass 0.176612671882913 -> 0.176612671716239
- link base_link: mass 0.725732279372378 -> 0.725732275378994
Joints:
- joint joint1: axis 0 0 1 -> 0 0 -1
- joint joint3: axis 0 0 1 -> 0 0 -1
- joint joint5: axis 0 0 1 -> 0 0 -1
- joint joint7: axis 0 0 1 -> 0 0 -1

File: rm_description/urdf/GEN72/rm_gen72.urdf.xacro (robot description, xacro)
@@ -46,22 +46,19 @@
     <xacro:Box_inertial_matrix m="500" l="1" w="1" h="0.02"/>
   </link>
-<!-- <?xml version="1.0" encoding="utf-8"?> -->
-<!-- <robot
-  name="GEN72"> -->
   <link
     name="base_link">
     <inertial>
       <origin
-        xyz="0.000608631599864255 0.000101410841221341 0.0500536423028978"
-        rpy="0 0 0" />
-      <mass
-        value="0.725732279372221" />
-      <inertia
-        ixx="0.00116526259312757"
-        ixy="3.86984764040053E-06"
-        ixz="3.61598634195252E-05"
-        iyy="0.00114387939249157"
-        iyz="-1.69159565748577E-06"
-        izz="0.000799620765266164" />
+        xyz="0.000608631901818564 0.000101410726070973 0.0500536421991602"
+        rpy="0 0 0" />
+      <mass
+        value="0.725732275378994" />
+      <inertia
+        ixx="0.00116526259423606"
+        ixy="3.86984316704955E-06"
+        ixz="3.61598587634246E-05"
+        iyy="0.00114387938317596"
+        iyz="-1.69159329895203E-06"
+        izz="0.000799620751622038" />
     </inertial>
     <visual>
@@ -93,15 +90,15 @@
     <inertial>
       <origin
-        xyz="3.54241616239891E-07 -6.04073277655109E-05 -0.0474562076947793"
-        rpy="0 0 0" />
-      <mass
-        value="0.511231576042974" />
-      <inertia
-        ixx="0.000959440501675413"
-        ixy="-1.90967914521654E-09"
-        ixz="-7.95751539476966E-09"
-        iyy="0.00102039305288465"
-        iyz="1.46570590325123E-06"
-        izz="0.000388714616194907" />
+        xyz="3.52736919702029E-07 -6.04059891453142E-05 -0.0474562080382229"
+        rpy="0 0 0" />
+      <mass
+        value="0.511231574249026" />
+      <inertia
+        ixx="0.000959440498156717"
+        ixy="-1.91894958276915E-09"
+        ixz="-7.95162454105223E-09"
+        iyy="0.00102039305580009"
+        iyz="1.46570350841548E-06"
+        izz="0.000388714614553318" />
     </inertial>
     <visual>
@@ -140,5 +137,5 @@
       link="Link1" />
     <axis
-      xyz="0 0 1" />
+      xyz="0 0 -1" />
     <limit
       lower="-3.0014"
@@ -151,15 +148,15 @@
     <inertial>
       <origin
-        xyz="-7.13241796657627E-07 -0.0576246216952895 -3.88440270542586E-05"
-        rpy="0 0 0" />
-      <mass
-        value="0.551907023014854" />
-      <inertia
-        ixx="0.00142140348660694"
-        ixy="-1.11761928109077E-08"
-        ixz="1.36372804172861E-08"
-        iyy="0.000525714272398651"
-        iyz="1.30499471806307E-06"
-        izz="0.00127234961251408" />
+        xyz="-7.11112352596068E-07 -0.0576246199640847 -3.88448280838247E-05"
+        rpy="0 0 0" />
+      <mass
+        value="0.551907049708684" />
+      <inertia
+        ixx="0.00142140355638731"
+        ixy="-1.11238202743335E-08"
+        ixz="1.36442937553009E-08"
+        iyy="0.000525714318152211"
+        iyz="1.30499854599536E-06"
+        izz="0.00127234964264819" />
     </inertial>
     <visual>
@@ -209,15 +206,15 @@
     <inertial>
       <origin
-        xyz="0.00897441376214199 2.62633968732563E-05 -0.0738284702130494"
-        rpy="0 0 0" />
-      <mass
-        value="0.774130450031732" />
-      <inertia
-        ixx="0.00242102073961797"
-        ixy="-6.22596416744622E-07"
-        ixz="-0.000489521447339777"
-        iyy="0.00248694314969316"
-        iyz="-1.4854289556066E-06"
-        izz="0.00090099718971981" />
+        xyz="0.00897441808005477 2.62636660835183E-05 -0.0738284677079453"
+        rpy="0 0 0" />
+      <mass
+        value="0.774130504869361" />
+      <inertia
+        ixx="0.00242102089342123"
+        ixy="-6.22567011177705E-07"
+        ixz="-0.000489521698616636"
+        iyy="0.00248694348279809"
+        iyz="-1.48555517772802E-06"
+        izz="0.000900997447038447" />
     </inertial>
     <visual>
@@ -256,5 +253,5 @@
       link="Link3" />
     <axis
-      xyz="0 0 1" />
+      xyz="0 0 -1" />
     <limit
       lower="-3.0014"
@@ -267,15 +264,15 @@
     <inertial>
       <origin
-        xyz="-0.0096243903445302 0.0352034287339325 0.000174576348464232"
-        rpy="0 0 0" />
-      <mass
-        value="0.437130215853835" />
-      <inertia
-        ixx="0.000866914153248166"
-        ixy="0.000148761646913658"
-        ixz="-7.42553547350131E-07"
-        iyy="0.000267753002587664"
-        iyz="2.6805826548563E-06"
-        izz="0.000952324298928138" />
+        xyz="-0.00962439034462223 0.0352034284437733 0.000174576348458631"
+        rpy="0 0 0" />
+      <mass
+        value="0.437130215851277" />
+      <inertia
+        ixx="0.000866914153243563"
+        ixy="0.000148761646911636"
+        ixz="-7.42553547115028E-07"
+        iyy="0.000267753002586622"
+        iyz="2.68058265443959E-06"
+        izz="0.000952324298922687" />
     </inertial>
     <visual>
@@ -325,15 +322,15 @@
     <inertial>
       <origin
-        xyz="-4.79650184286029E-07 -3.84737693792612E-05 -0.0669554878200541"
-        rpy="0 0 0" />
-      <mass
-        value="0.424276753764529" />
-      <inertia
-        ixx="0.0011244489011316"
-        ixy="7.56623220194193E-09"
-        ixz="-1.71276249932631E-08"
-        iyy="0.00103382374928123"
-        iyz="8.2469441747875E-07"
-        izz="0.000274640088277484" />
+        xyz="-4.79650184265212E-07 -3.84737693796814E-05 -0.0669554881104284"
+        rpy="0 0 0" />
+      <mass
+        value="0.424276753764533" />
+      <inertia
+        ixx="0.00112444890113163"
+        ixy="7.56623220322765E-09"
+        ixz="-1.71276249952398E-08"
+        iyy="0.00103382374928125"
+        iyz="8.24694417490181E-07"
+        izz="0.000274640088277489" />
     </inertial>
     <visual>
@@ -372,121 +369,5 @@
       link="Link5" />
     <axis
-      xyz="0 0 1" />
-    <limit
-      lower="-3.0014"
-      upper="3.0014"
-      effort="5"
-      velocity="3.141" />
-  </joint>
-  <link
-    name="Link6">
-    <inertial>
-      <origin
-        xyz="0.00184221691932426 0.0379763265035087 -9.21090904324274E-05"
-        rpy="0 0 0" />
-      <mass
-        value="0.302793039332829" />
-      <inertia
-        ixx="0.00014011480503376"
-        ixy="-3.00204828273403E-06"
-        ixz="-4.58155498967514E-10"
-        iyy="0.000132631402640971"
-        iyz="7.01344540252765E-10"
-        izz="0.000155721320872423" />
-    </inertial>
-    <visual>
-      <origin
-        xyz="0 0 0"
-        rpy="0 0 0" />
-      <geometry>
-        <mesh
-          filename="package://rm_description/meshes/GEN72/Link6.STL" />
-      </geometry>
-      <material
-        name="">
-        <color
-          rgba="1 1 1 1" />
-      </material>
-    </visual>
-    <collision>
-      <origin
-        xyz="0 0 0"
-        rpy="0 0 0" />
-      <geometry>
-        <mesh
-          filename="package://rm_description/meshes/GEN72/Link6.STL" />
-      </geometry>
-    </collision>
-  </link>
-  <joint
-    name="joint6"
-    type="revolute">
-    <origin
-      xyz="0 0 0"
-      rpy="1.5708 0 0" />
-    <parent
-      link="Link5" />
-    <child
-      link="Link6" />
-    <axis
-      xyz="0 0 1" />
-    <limit
-      lower="-1.707"
-      upper="1.783"
-      effort="5"
-      velocity="3.141" />
-  </joint>
-  <link
-    name="Link7">
-    <inertial>
-      <origin
-        xyz="0.000199884675729955 -4.25081843764018E-08 -0.0292498694019246"
-        rpy="0 0 0" />
-      <mass
-        value="0.176612671882913" />
-      <inertia
-        ixx="6.24281233883421E-05"
-        ixy="2.55814128580721E-10"
-        ixz="-3.1014379202721E-12"
-        iyy="6.24291486534025E-05"
-        iyz="1.37181281239386E-11"
-        izz="8.48642555354654E-05" />
-    </inertial>
-    <visual>
-      <origin
-        xyz="0 0 0"
-        rpy="0 0 0" />
-      <geometry>
-        <mesh
-          filename="package://rm_description/meshes/GEN72/Link7.STL" />
-      </geometry>
-      <material
-        name="">
-        <color
-          rgba="1 1 1 1" />
-      </material>
-    </visual>
-    <collision>
-      <origin
-        xyz="0 0 0"
-        rpy="0 0 0" />
-      <geometry>
-        <mesh
-          filename="package://rm_description/meshes/GEN72/Link7.STL" />
-      </geometry>
-    </collision>
-  </link>
-  <joint
-    name="joint7"
-    type="revolute">
-    <origin
-      xyz="0.0905 0.067 0"
-      rpy="1.5708 0 1.5708" />
-    <parent
-      link="Link6" />
-    <child
-      link="Link7" />
-    <axis
-      xyz="0 0 1" />
+      xyz="0 0 -1" />
     <limit
       lower="-3.0014"
@@ -495,5 +376,121 @@
       velocity="3.926" />
   </joint>
-    <!-- Transmissions for ROS Control -->
+  <link
+    name="Link6">
+    <inertial>
+      <origin
+        xyz="0.00184221175785321 0.0379763273402476 -9.2109082789162E-05"
+        rpy="0 0 0" />
+      <mass
+        value="0.302793071336592" />
+      <inertia
+        ixx="0.000140114798143356"
+        ixy="-3.0020621302762E-06"
+        ixz="-4.58156507440607E-10"
+        iyy="0.000132631412915026"
+        iyz="7.01344406582159E-10"
+        izz="0.000155721318559448" />
+    </inertial>
+    <visual>
+      <origin
+        xyz="0 0 0"
+        rpy="0 0 0" />
+      <geometry>
+        <mesh
+          filename="package://rm_description/meshes/GEN72/Link6.STL" />
+      </geometry>
+      <material
+        name="">
+        <color
+          rgba="1 1 1 1" />
+      </material>
+    </visual>
+    <collision>
+      <origin
+        xyz="0 0 0"
+        rpy="0 0 0" />
+      <geometry>
+        <mesh
+          filename="package://rm_description/meshes/GEN72/Link6.STL" />
+      </geometry>
+    </collision>
+  </link>
+  <joint
+    name="joint6"
+    type="revolute">
+    <origin
+      xyz="0 0 0"
+      rpy="1.5708 0 0" />
+    <parent
+      link="Link5" />
+    <child
+      link="Link6" />
+    <axis
+      xyz="0 0 1" />
+    <limit
+      lower="-1.707"
+      upper="1.783"
+      effort="5"
+      velocity="3.926" />
+  </joint>
+  <link
+    name="Link7">
+    <inertial>
+      <origin
+        xyz="0.000200062483601049 1.38702560039998E-08 -0.0292498560100851"
+        rpy="0 0 0" />
+      <mass
+        value="0.176612671716239" />
+      <inertia
+        ixx="6.24286469682688E-05"
+        ixy="5.70592007031404E-10"
+        ixz="-4.73833817662725E-11"
+        iyy="6.24286273697226E-05"
+        iyz="-4.26919211524294E-11"
+        izz="8.48642578603026E-05" />
+    </inertial>
+    <visual>
+      <origin
+        xyz="0 0 0"
+        rpy="0 0 0" />
+      <geometry>
+        <mesh
+          filename="package://rm_description/meshes/GEN72/Link7.STL" />
+      </geometry>
+      <material
+        name="">
+        <color
+          rgba="1 1 1 1" />
+      </material>
+    </visual>
+    <collision>
+      <origin
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