Commit message: doc:添加一体化六维力适配，添加控制器1.6.7适配，添加UDP控制功能适配

File: rm_description/urdf/RML63/rml_63_bottom.urdf.xacro (robot description, xacro)
@@ -54,15 +54,15 @@
     <inertial>
       <origin
-        xyz="0.0014231 -0.00010178 0.050147"
-        rpy="0 0 0" />
-      <mass
-        value="0.66171" />
-      <inertia
-        ixx="0.00099443"
-        ixy="3.282E-06"
-        ixz="-9.9964E-06"
-        iyy="0.0010144"
-        iyz="1.2811E-06"
-        izz="0.00067929" />
+        xyz="0.0002051 -8.259E-05 0.043092"
+        rpy="0 0 0" />
+      <mass
+        value="1.6314" />
+      <inertia
+        ixx="0.0022252"
+        ixy="7.9005E-06"
+        ixz="-7.7558E-05"
+        iyy="0.0022156"
+        iyz="5.9846E-06"
+        izz="0.0018513" />
     </inertial>
     <visual>
@@ -77,4 +77,44 @@
         name="">
         <color
+          rgba="0.86667 0.86667 0.8902 1" />
+      </material>
+    </visual>
+    <collision>
+      <origin
+        xyz="0 0 0"
+        rpy="0 0 0" />
+      <geometry>
+        <mesh
+          filename="package://rm_description/meshes/RML63/base_link.STL" />
+      </geometry>
+    </collision>
+  </link>
+  <link
+    name="link1">
+    <inertial>
+      <origin
+        xyz="-0.030909 -0.0013023 -0.0053121"
+        rpy="0 0 0" />
+      <mass
+        value="1.7668" />
+      <inertia
+        ixx="0.0014534"
+        ixy="-0.00017578"
+        ixz="0.0002802"
+        iyy="0.0043772"
+        iyz="1.7209E-05"
+        izz="0.0040911" />
+    </inertial>
+    <visual>
+      <origin
+        xyz="0 0 0"
+        rpy="0 0 0" />
+      <geometry>
+        <mesh
+          filename="package://rm_description/meshes/RML63/link1.STL" />
+      </geometry>
+      <material
+        name="">
+        <color
           rgba="1 1 1 1" />
       </material>
@@ -86,46 +126,6 @@
       <geometry>
         <mesh
-          filename="package://rm_description/meshes/RML63/base_link.STL" />
-      </geometry>
-    </collision>
-  </link>
-  <link
-    name="link1">
-    <inertial>
-      <origin
-        xyz="-0.043281 -0.0072256 -0.012694"
-        rpy="0 0 0" />
-      <mass
-        value="0.89496" />
-      <inertia
-        ixx="0.0010156"
-        ixy="-0.00026764"
-        ixz="0.00045014"
-        iyy="0.0024107"
-        iyz="6.0996E-05"
-        izz="0.0022755" />
-    </inertial>
-    <visual>
-      <origin
-        xyz="0 0 0"
-        rpy="0 0 0" />
-      <geometry>
-        <mesh
           filename="package://rm_description/meshes/RML63/link1.STL" />
       </geometry>
-      <material
-        name="">
-        <color
-          rgba="1 1 1 1" />
-      </material>
-    </visual>
-    <collision>
-      <origin
-        xyz="0 0 0"
-        rpy="0 0 0" />
-      <geometry>
-        <mesh
-          filename="package://rm_description/meshes/RML63/link1.STL" />
-      </geometry>
     </collision>
   </link>
@@ -134,5 +134,5 @@
     type="revolute">
     <origin
-      xyz="0 0 0.172"
+      xyz="0 0 0.1625"
       rpy="0 0 0" />
     <parent
@@ -141,191 +141,191 @@
       link="link1" />
     <axis
+      xyz="0 0 -1" />
+    <limit
+      lower="-3.107"
+      upper="3.107"
+      effort="100"
+      velocity="1" />
+    <dynamics
+      damping="50"
+      friction="1" />
+  </joint>
+  <link
+    name="link2">
+    <inertial>
+      <origin
+        xyz="0.16852 9.8217E-07 -0.077258"
+        rpy="0 0 0" />
+      <mass
+        value="4.3415" />
+      <inertia
+        ixx="0.0028306"
+        ixy="3.3846E-07"
+        ixz="4.0484E-06"
+        iyy="0.075435"
+        iyz="-3.3974E-08"
+        izz="0.075923" />
+    </inertial>
+    <visual>
+      <origin
+        xyz="0 0 0"
+        rpy="0 0 0" />
+      <geometry>
+        <mesh
+          filename="package://rm_description/meshes/RML63/link2.STL" />
+      </geometry>
+      <material
+        name="">
+        <color
+          rgba="0.86667 0.86667 0.8902 1" />
+      </material>
+    </visual>
+    <collision>
+      <origin
+        xyz="0 0 0"
+        rpy="0 0 0" />
+      <geometry>
+        <mesh
+          filename="package://rm_description/meshes/RML63/link2.STL" />
+      </geometry>
+    </collision>
+  </link>
+  <joint
+    name="joint2"
+    type="revolute">
+    <origin
+      xyz="-0.086 0 0"
+      rpy="-1.5708 -1.5708 0" />
+    <parent
+      link="link1" />
+    <child
+      link="link2" />
+    <axis
       xyz="0 0 1" />
     <limit
-      lower="-3.106"
-      upper="3.106"
-      effort="100"
-      velocity="1" />
-    <dynamics
-      damping="50"
-      friction="1" />
-  </joint>
-  <link
-    name="link2">
-    <inertial>
-      <origin
-        xyz="0.17388 3.639E-07 -0.089966"
-        rpy="0 0 0" />
-      <mass
-        value="1.5679" />
-      <inertia
-        ixx="0.0010615"
-        ixy="-7.3371E-08"
-        ixz="-0.00025488"
-        iyy="0.03035"
-        iyz="-1.6148E-08"
-        izz="0.030485" />
-    </inertial>
-    <visual>
-      <origin
-        xyz="0 0 0"
-        rpy="0 0 0" />
-      <geometry>
-        <mesh
-          filename="package://rm_description/meshes/RML63/link2.STL" />
-      </geometry>
-      <material
-        name="">
-        <color
-          rgba="1 1 1 1" />
-      </material>
-    </visual>
-    <collision>
-      <origin
-        xyz="0 0 0"
-        rpy="0 0 0" />
-      <geometry>
-        <mesh
-          filename="package://rm_description/meshes/RML63/link2.STL" />
-      </geometry>
-    </collision>
-  </link>
-  <joint
-    name="joint2"
-    type="revolute">
-    <origin
-      xyz="-0.086 0 0"
-      rpy="0 -1.5708 -1.5708" />
-    <parent
-      link="link1" />
-    <child
+      lower="-3.107"
+      upper="3.107"
+      effort="100"
+      velocity="1" />
+    <dynamics
+      damping="50"
+      friction="1" />
+  </joint>
+  <link
+    name="link3">
+    <inertial>
+      <origin
+        xyz="0.034488 -0.010948 -0.0056239"
+        rpy="0 0 0" />
+      <mass
+        value="1.7286" />
+      <inertia
+        ixx="0.0014154"
+        ixy="0.00068025"
+        ixz="-0.00043307"
+        iyy="0.0026049"
+        iyz="0.00017201"
+        izz="0.0028551" />
+    </inertial>
+    <visual>
+      <origin
+        xyz="0 0 0"
+        rpy="0 0 0" />
+      <geometry>
+        <mesh
+          filename="package://rm_description/meshes/RML63/link3.STL" />
+      </geometry>
+      <material
+        name="">
+        <color
+          rgba="0.86667 0.86667 0.8902 1" />
+      </material>
+    </visual>
+    <collision>
+      <origin
+        xyz="0 0 0"
+        rpy="0 0 0" />
+      <geometry>
+        <mesh
+          filename="package://rm_description/meshes/RML63/link3.STL" />
+      </geometry>
+    </collision>
+  </link>
+  <joint
+    name="joint3"
+    type="revolute">
+    <origin
+      xyz="0.38 0 0"
+      rpy="0 0 1.5708" />
+    <parent
       link="link2" />
+    <child
+      link="link3" />
     <axis
       xyz="0 0 1" />
     <limit
-      lower="-3.106"
-      upper="3.106"
-      effort="100"
-      velocity="1" />
-    <dynamics
-      damping="50"
-      friction="1" />
-  </joint>
-  <link
-    name="link3">
-    <inertial>
-      <origin
-        xyz="0.035968 -0.020568 -0.0048526"
-        rpy="0 0 0" />
-      <mass
-        value="0.67539" />
-      <inertia
-        ixx="0.00091144"
-        ixy="0.00043238"
-        ixz="-0.0001205"
-        iyy="0.0012128"
-        iyz="6.6376E-05"
-        izz="0.0015231" />
-    </inertial>
-    <visual>
-      <origin
-        xyz="0 0 0"
-        rpy="0 0 0" />
-      <geometry>
-        <mesh
-          filename="package://rm_description/meshes/RML63/link3.STL" />
-      </geometry>
-      <material
-        name="">
-        <color
-          rgba="1 1 1 1" />
-      </material>
-    </visual>
-    <collision>
-      <origin
-        xyz="0 0 0"
-        rpy="0 0 0" />
-      <geometry>
-        <mesh
-          filename="package://rm_description/meshes/RML63/link3.STL" />
-      </geometry>
-    </collision>
-  </link>
-  <joint
-    name="joint3"
-    type="revolute">
-    <origin
-      xyz="0.38 0 -0.00030011"
-      rpy="0 0 1.5708" />
-    <parent
-      link="link2" />
-    <child
+      lower="-3.107"
+      upper="2.531"
+      effort="100"
+      velocity="1" />
+    <dynamics
+      damping="50"
+      friction="1" />
+  </joint>
+  <link
+    name="link4">
+    <inertial>
+      <origin
+        xyz="4.1778E-07 -0.030483 -0.19739"
+        rpy="0 0 0" />
+      <mass
+        value="2.4734" />
+      <inertia
+        ixx="0.02602"
+        ixy="-1.1659E-07"
+        ixz="3.1323E-07"
+        iyy="0.024375"
+        iyz="0.0061661"
+        izz="0.002958" />
+    </inertial>
+    <visual>
+      <origin
+        xyz="0 0 0"
+        rpy="0 0 0" />
+      <geometry>
+        <mesh
+          filename="package://rm_description/meshes/RML63/link4.STL" />
+      </geometry>
+      <material
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
File: rm_description/urdf/RML63/rml_63_description.urdf (robot description, URDF)
Before this commit: robot rml_63_description, 7 links, 6 joints
Links:
- link base_link: mass 0.66171 -> 1.6314
- link link1: mass 0.89496 -> 1.7668
- link link2: mass 1.5679 -> 4.3415
- link link3: mass 0.67539 -> 1.7286
- link link4: mass 0.69687 -> 2.4734
- link link5: mass 0.34759 -> 0.93162
- link link6: mass 0.077104 -> 0.065037
Joints:
- joint joint1: axis 0 0 1 -> 0 0 -1; limit lower=-3.106 upper=3.106 effort=100 velocity=1 -> lower=-3.107 upper=3.107 effort=100 velocity=1; origin xyz=0 0 0.172 rpy=0 0 0 -> xyz=0 0 0.1625 rpy=0 0 0
- joint joint2: limit lower=-3.106 upper=3.106 effort=100 velocity=1 -> lower=-3.107 upper=3.107 effort=100 velocity=1; origin xyz=-0.086 0 0 rpy=0 -1.5708 -1.5708 -> xyz=-0.086 0 0 rpy=-1.5708 -1.5708 0
- joint joint3: limit lower=-3.106 upper=2.53 effort=100 velocity=1 -> lower=-3.107 upper=2.531 effort=100 velocity=1; origin xyz=0.38 0 -0.00030011 rpy=0 0 1.5708 -> xyz=0.38 0 0 rpy=0 0 1.5708
- joint joint4: axis 0 0 1 -> 0 0 -1; limit lower=-3.106 upper=3.106 effort=100 velocity=1 -> lower=-3.107 upper=3.107 effort=100 velocity=1; origin xyz=0.069 -0.405 0.00029958 rpy=1.5708 0 0 -> xyz=0.069 -0.405 0 rpy=1.5708 0 0
- joint joint5: axis 0 0 1 -> 0 0 -1; limit lower=-3.106 upper=3.106 effort=100 velocity=1 -> lower=-3.107 upper=3.107 effort=100 velocity=1
- joint joint6: axis 0 0 1 -> 0 0 -1; limit lower=-6.28 upper=6.28 effort=100 velocity=1 -> lower=-3.14 upper=3.14 effort=100 velocity=1; origin xyz=0 0.115 0 rpy=1.5708 0 3.1416 -> xyz=-0.00010308 0.115 -0.00010734 rpy=1.5708 0 3.1416

Commit message: feat: 新增接口并适配三代四代控制器

File: rm_description/urdf/ECO63/eco63.urdf (robot description, URDF)
Before this commit: robot rm_eco63, 7 links, 6 joints
Joints:
- joint joint1: axis 0 0 1 -> 0 0 -1

File: rm_description/urdf/RML63/rml_63_description.urdf (robot description, URDF)
Before this commit: robot rml_63_description, 7 links, 6 joints
Joints:
- joint joint1: axis 0 0 -1 -> 0 0 1
- joint joint4: axis 0 0 -1 -> 0 0 1
- joint joint5: axis 0 0 -1 -> 0 0 1
- joint joint6: axis 0 0 -1 -> 0 0 1
