Commit message: doc:fix gen72urdf error

File: rm_description/urdf/GEN72/GEN72.urdf (robot description, URDF)
Before this commit: robot GEN72, 8 links, 7 joints
Joints:
- joint joint7: origin xyz=0.0742 0.067 0 rpy=0 0 1.5708 -> xyz=0.0742 0.067 0 rpy=1.5708 0 1.5708

File: rm_description/urdf/GEN72/rm_gen72.urdf.xacro (robot description, xacro)
@@ -441,5 +441,5 @@
     <inertial>
       <origin
-        xyz="0.000199885014846801 0.0211000079719058 -4.90848725240361E-08"
+        xyz="0.000199885014846801 -4.90848725240361E-08 -0.0211000079719058"
         rpy="0 0 0" />
       <mass
@@ -447,9 +447,9 @@
       <inertia
         ixx="4.95156474993269E-05"
-        ixy="3.10143792228514E-12"
-        ixz="2.55814128583062E-10"
-        iyy="6.12184422048225E-05"
-        iyz="-1.37181281244006E-11"
-        izz="4.95166727643872E-05" />
+        ixy="2.55814128582907E-10"
+        ixz="-3.10143792187155E-12"
+        iyy="4.95166727643872E-05"
+        iyz="1.37181281241938E-11"
+        izz="6.12184422048225E-05" />
     </inertial>
     <visual>
@@ -482,5 +482,5 @@
     <origin
       xyz="0.0742 0.067 0"
-      rpy="0 0 1.5708" />
+      rpy="1.5708 0 1.5708" />
     <parent
       link="Link6" />

Commit message: doc:fix gen72 moveit error

File: rm_description/urdf/GEN72/GEN72.urdf (robot description, URDF)
Before this commit: robot GEN72, 8 links, 7 joints
Joints:
- joint joint7: axis 0 1 0 -> 0 0 1

File: rm_description/urdf/GEN72/rm_gen72.urdf.xacro (robot description, xacro)
@@ -488,5 +488,5 @@
       link="Link7" />
     <axis
-      xyz="0 1 0" />
+      xyz="0 0 1" />
     <limit
       lower="-3.0014"

Commit message: doc:fix gen72 urdf error

File: rm_description/urdf/GEN72/GEN72.urdf (robot description, URDF)
Before this commit: robot GEN72, 8 links, 7 joints
Links:
- link Link3: mass 0.774130450031732 -> 0.774130450031718
- link Link4: mass 0.437130215853835 -> 0.437130215853825
- link Link7: mass 0.127401822079286 -> 0.176612671882913
- link base_link: mass 0.725732279372221 -> 0.725732279372378
Joints:
- joint joint5: limit lower=-3.0014 upper=3.0014 effort=5 velocity=3.141 -> lower=-3.0014 upper=3.0014 effort=5 velocity=3.926
- joint joint6: limit lower=-1.707 upper=1.783 effort=5 velocity=3.141 -> lower=-1.707 upper=1.783 effort=5 velocity=3.926
- joint joint7: limit lower=-3.0014 upper=3.0014 effort=5 velocity=3.141 -> lower=-3.0014 upper=3.0014 effort=5 velocity=3.926; origin xyz=0.0742 0.067 0 rpy=1.5708 0 1.5708 -> xyz=0.0905 0.067 0 rpy=1.5708 0 1.5708

File: rm_description/urdf/GEN72/rm_gen72.urdf.xacro (robot description, xacro)
@@ -441,15 +441,15 @@
     <inertial>
       <origin
-        xyz="0.000199885014846801 -4.90848725240361E-08 -0.0211000079719058"
-        rpy="0 0 0" />
-      <mass
-        value="0.127401822079286" />
-      <inertia
-        ixx="4.95156474993269E-05"
-        ixy="2.55814128582907E-10"
-        ixz="-3.10143792187155E-12"
-        iyy="4.95166727643872E-05"
-        iyz="1.37181281241938E-11"
-        izz="6.12184422048225E-05" />
+        xyz="0.000199884675729955 -4.25081843764018E-08 -0.0292498694019246"
+        rpy="0 0 0" />
+      <mass
+        value="0.176612671882913" />
+      <inertia
+        ixx="6.24281233883421E-05"
+        ixy="2.55814128580721E-10"
+        ixz="-3.1014379202721E-12"
+        iyy="6.24291486534025E-05"
+        iyz="1.37181281239386E-11"
+        izz="8.48642555354654E-05" />
     </inertial>
     <visual>
@@ -481,5 +481,5 @@
     type="revolute">
     <origin
-      xyz="0.0742 0.067 0"
+      xyz="0.0905 0.067 0"
       rpy="1.5708 0 1.5708" />
     <parent
@@ -493,5 +493,5 @@
       upper="3.0014"
       effort="5"
-      velocity="3.141" />
+      velocity="3.926" />
   </joint>
     <!-- Transmissions for ROS Control -->
